Commit message: 0731

File: controllers/controller_test_path_try_fix_arm/LRMate-200iD_try_fix_arm_itri.urdf (robot description, URDF)
Before this commit: robot LRMate-200iD, 1 links, 0 joints
Links:
- added link J1, mass 14.3548583797231; collision mesh filename=package://stl/J2BASE_UNIT_0.001.stl; visual mesh filename=package://stl/J1BASE_UNIT_0.001.stl
Joints:
- added joint J1: type revolute, parent Base, child J1, origin xyz=0 0 0.169 rpy=0 0 0, axis 0 0 1, limit lower=-2.9671 upper=2.9671 effort=0 velocity=0
